Commit message: new

File: src/bobac3_description/xacro/bobac3_base.xacro (robot description, xacro)
@@ -12,17 +12,17 @@
         <origin xyz="0.0 0.0 0.0" rpy="0.0 0.0 0.0" />
         <geometry>
-          <cylinder radius="0.12" length="0.025" />
+          <cylinder radius="0.001" length="0.001" />
         </geometry>
         <material name="LightGrey">
-          <color rgba="1.0 1.0 1.0 1.0" />
-        </material>
-      </visual>
-      <collision>
-        <geometry>
-          <cylinder radius="0.12" length="0.025" />
-        </geometry>
-      </collision>
-      <inertial>
-        <mass value="5.0" />
+          <color rgba="1.0 1.0 1.0 0.0" />
+        </material>
+      </visual>
+      <collision>
+        <geometry>
+          <cylinder radius="0.15" length="0.01" />
+        </geometry>
+      </collision>
+      <inertial>
+        <mass value="500.0" />
         <origin xyz="0.0 0.0 0.0" rpy="0.0 0.0 0.0" />
         <inertia ixx="3.0" ixy="0.0" ixz="0.0" iyy="3.0" iyz="0.0" izz="3.0" />
@@ -32,8 +32,32 @@
       <!-- xyz="0.0 0 0.03" -->
       <origin
-        xyz="0.0 0 0.0125"
+        xyz="0.0 0 0.005"
         rpy="0 0 0" />
       <parent link="base_footprint" />
       <child link="base_link" />
+    </joint>
+    <link name="charge_port_link">
+      <visual>
+        <origin xyz="0.0 0.0 0.0" rpy="0.0 0.0 0.0" />
+        <geometry>
+          <box size="0.03 0.02 0.005" />
+        </geometry>
+        <material name="charge_left">
+          <color rgba="1.0 0.5 0.0 1.0" />
+        </material>
+      </visual>
+      <collision>
+        <geometry>
+           <box size="0.03 0.02 0.005" />
+        </geometry>
+      </collision>
+    </link>
+    <joint name="base_charge_joint" type="fixed">
+      <!-- xyz="0.0 0 0.03" -->
+      <origin
+        xyz="-0.16 0.0 -0.0075"
+        rpy="0 0 0" />
+      <parent link="base_link" />
+      <child link="charge_port_link" />
     </joint>
     <link
@@ -341,4 +365,10 @@
       <axis
         xyz="0 0 0" />
+    </joint>
+    <link name="bottom_camera_optical_link" />
+    <joint name="bottom_camera_optical_joint" type="fixed">
+      <parent link="bottom_camera_link" />
+      <child link="bottom_camera_optical_link" />
+      <origin xyz="0 0 0" rpy="-1.57079 0 -1.57079" />
     </joint>
     <link

File: src/bobac3_description/xacro/gazebo_plugin.xacro (robot description, xacro)
@@ -11,11 +11,16 @@
       </plugin>
     </gazebo>
+    <gazebo reference="charge_port_link">
+      <material>Gazebo/Orange</material>
+    </gazebo>
     <gazebo reference="base_footprint">
       <material>Gazebo/GreyTransparent</material>
+      <mu1>0.0</mu1>
+      <mu2>0.0</mu2>
     </gazebo>
     <gazebo reference="base_link">
       <material>Gazebo/White</material>
     </gazebo>
-    <gazebo reference="humtemper_link">
+    <gazebo reference="humtmper_link">
       <material>Gazebo/FlatBlack</material>
     </gazebo>
@@ -29,5 +34,5 @@
       <material>Gazebo/FlatBlack</material>
     </gazebo>
-    <gazebo reference="smoke_sensor_link">
+    <gazebo reference="smoke_link">
       <material>Gazebo/FlatBlack</material>
     </gazebo>
@@ -43,4 +48,19 @@
     <gazebo reference="base_depth_link">
       <material>Gazebo/FlatBlack</material>
+    </gazebo>
+    <gazebo reference="left/wheel_link">
+      <material>Gazebo/FlatBlack</material>
+      <mu1>0.0</mu1>
+      <mu2>0.0</mu2>
+    </gazebo>
+    <gazebo reference="right/wheel_link">
+      <material>Gazebo/FlatBlack</material>
+      <mu1>0.0</mu1>
+      <mu2>0.0</mu2>
+    </gazebo>
+    <gazebo reference="front/wheel_link">
+      <material>Gazebo/FlatBlack</material>
+      <mu1>0.0</mu1>
+      <mu2>0.0</mu2>
     </gazebo>
     <gazebo reference="fuse_lidar_link">
@@ -61,5 +81,5 @@
           <range>
             <min>0.15</min>
-            <max>30.0</max>
+            <max>10.0</max>
             <resolution>0.01</resolution>
           </range>
@@ -110,5 +130,5 @@
           <imageTopicName>image_raw</imageTopicName>
           <cameraInfoTopicName>camera_info</cameraInfoTopicName>
-          <frameName>bottom_camera_link</frameName>
+          <frameName>bottom_camera_optical_link</frameName>
           <hackBaseline>0.07</hackBaseline>
           <distortionK1>0.0</distortionK1>
