Commit message: awdwa

File: src/bobac3_description/xacro/basic_kit.xacro (robot description, xacro)
@@ -1,93 +1,193 @@
 <?xml version="1.0"?>
 <robot xmlns:xacro="http://www.ros.org/wiki/xacro" name="basic_kit">
-  <xacro:macro name="basic_kit" params="parent xyz rpy sim">
+  <xacro:macro name="basic_kit" params="parent sim laser_type">
     <joint name="extra_kit_joint" type="fixed">
       <parent link="${parent}" />
       <child link="basic_kit_link" />
-      <origin xyz="${xyz}" rpy="${rpy}" />
+      <xacro:if value="${laser_type == 'CSPC'}">
+        <origin xyz="-0.199 0 -0.02" rpy="0 0 0" />
+      </xacro:if>
+      <xacro:unless value="${laser_type == 'CSPC'}">
+        <origin xyz="-0.034 0 0" rpy="0 0 0" />
+      </xacro:unless>
       <axis xyz="0 0 0" />
     </joint>
-    <link name="basic_kit_link">
-      <inertial>
+    <xacro:if value="${laser_type == 'CSPC'}">
+      <link
+        name="basic_kit_link">
+        <inertial>
+          <origin
+            xyz="-0.0911672576716816 -0.00375101667946967 0.327523997489668"
+            rpy="0 0 0" />
+          <mass
+            value="1.45911195846713" />
+          <inertia
+            ixx="0.0111746368285295"
+            ixy="6.02134621630998E-06"
+            ixz="-0.00136442928293414"
+            iyy="0.00566215613507705"
+            iyz="1.11054482788563E-05"
+            izz="0.0092111197679973" />
+        </inertial>
+        <visual>
+          <origin
+            xyz="0 0 0"
+            rpy="0 0 0" />
+          <geometry>
+            <mesh
+              filename="package://bobac3_description/meshes/basic_kit_link_cspc.STL" />
+          </geometry>
+          <material
+            name="">
+            <color
+              rgba="1 1 1 1" />
+          </material>
+        </visual>
+        <collision>
+          <origin
+            xyz="0 0 0"
+            rpy="0 0 0" />
+          <geometry>
+            <mesh
+              filename="package://bobac3_description/meshes/basic_kit_link_cspc.STL" />
+          </geometry>
+        </collision>
+      </link>
+    </xacro:if>
+    <xacro:unless value="${laser_type == 'CSPC'}">
+      <link name="basic_kit_link">
+        <inertial>
+          <origin
+            xyz="0.063843 0.001458 0.284233"
+            rpy="0 0 0" />
+          <mass
+            value="1.44666566726349" />
+          <inertia
+            ixx="0.0142506995251501"
+            ixy="-2.97587772816469E-07"
+            ixz="0.000982982938097122"
+            iyy="0.00748136009628222"
+            iyz="-1.45498390881542E-05"
+            izz="0.00855600296958952" />
+        </inertial>
+        <visual>
+          <origin
+            xyz="0 0 0"
+            rpy="0 0 0" />
+          <geometry>
+            <mesh
+              filename="package://bobac3_description/meshes/basic_kit_link.STL" />
+          </geometry>
+          <material
+            name="">
+            <color
+              rgba="1 1 1 1" />
+          </material>
+        </visual>
+        <collision>
+          <origin
+            xyz="0 0 0"
+            rpy="0 0 0" />
+          <geometry>
+            <mesh
+              filename="package://bobac3_description/meshes/basic_kit_link.STL" />
+          </geometry>
+        </collision>
+      </link>
+    </xacro:unless>
+    <xacro:if value="${laser_type == 'CSPC'}">
+      <link
+        name="top_camera_link">
+        <inertial>
+          <origin
+            xyz="-0.0144410472853577 3.50221192592643E-07 -0.0155879253099328"
+            rpy="0 0 0" />
+          <mass
+            value="0.0930702512999254" />
+          <inertia
+            ixx="8.46696104375507E-05"
+            ixy="1.7202977510131E-11"
+            ixz="1.4425416685427E-06"
+            iyy="5.8230348276419E-05"
+            iyz="-1.00759165191464E-10"
+            izz="3.74977551477733E-05" />
+        </inertial>
+        <visual>
+          <origin
+            xyz="0 0 0"
+            rpy="0 0 0" />
+          <geometry>
+            <mesh
+              filename="package://bobac3_description/meshes/top_camera_link.STL" />
+          </geometry>
+          <material
+            name="">
+            <color
+              rgba="1 1 1 1" />
+          </material>
+        </visual>
+        <collision>
+          <origin
+            xyz="0 0 0"
+            rpy="0 0 0" />
+          <geometry>
+            <mesh
+              filename="package://bobac3_description/meshes/top_camera_link.STL" />
+          </geometry>
+        </collision>
+      </link>
+    </xacro:if>
+    <xacro:unless value="${laser_type == 'CSPC'}">
+      <link name="top_camera_link">
+        <inertial>
+          <origin
+            xyz="-0.01444 0.0 -0.0155877"
+            rpy="0 0 0" />
+          <mass
+            value="0.0930723033732641" />
+          <inertia
+            ixx="8.46719406198911E-05"
+            ixy="1.72756831136607E-21"
+            ixz="1.44257463259852E-06"
+            iyy="5.82306984916293E-05"
+            iyz="8.09942701300137E-21"
+            izz="3.7499909854723E-05" />
+        </inertial>
+        <visual>
+          <origin
+            xyz="0 0 0"
+            rpy="0 0 0" />
+          <geometry>
+            <mesh
+              filename="package://bobac3_description/meshes/top_camera_link.STL" />
+          </geometry>
+          <material
+            name="">
+            <color
+              rgba="0.5 0.5 0.5 1" />
+          </material>
+        </visual>
+        <collision>
+          <origin
+            xyz="0 0 0"
+            rpy="0 0 0" />
+          <geometry>
+            <mesh
+              filename="package://bobac3_description/meshes/top_camera_link.STL" />
+          </geometry>
+        </collision>
+      </link>
+    </xacro:unless>
+    <joint name="top_camera_joint" type="fixed">
+      <xacro:if value="${laser_type == 'CSPC'}">
         <origin
-          xyz="0.063843 0.001458 0.284233"
-          rpy="0 0 0" />
-        <mass
-          value="1.44666566726349" />
-        <inertia
-          ixx="0.0142506995251501"
-          ixy="-2.97587772816469E-07"
-          ixz="0.000982982938097122"
-          iyy="0.00748136009628222"
-          iyz="-1.45498390881542E-05"
-          izz="0.00855600296958952" />
-      </inertial>
-      <visual>
+          xyz="-0.016389 0 0.45762"
+          rpy="0 -0.7854 3.1416" />
+      </xacro:if>
+      <xacro:unless value="${laser_type == 'CSPC'}">
         <origin
-          xyz="0 0 0"
-          rpy="0 0 0" />
-        <geometry>
-          <mesh
-            filename="package://bobac3_description/meshes/basic_kit_link.STL" />
-        </geometry>
-        <material
-          name="">
-          <color
-            rgba="1 1 1 1" />
-        </material>
-      </visual>
-      <collision>
-        <origin
-          xyz="0 0 0"
-          rpy="0 0 0" />
-        <geometry>
-          <mesh
-            filename="package://bobac3_description/meshes/basic_kit_link.STL" />
-        </geometry>
-      </collision>
-    </link>
-    <link name="top_camera_link">
-      <inertial>
-        <origin
-          xyz="-0.01444 0.0 -0.0155877"
-          rpy="0 0 0" />
-        <mass
-          value="0.0930723033732641" />
-        <inertia
-          ixx="8.46719406198911E-05"
-          ixy="1.72756831136607E-21"
-          ixz="1.44257463259852E-06"
-          iyy="5.82306984916293E-05"
-          iyz="8.09942701300137E-21"
-          izz="3.7499909854723E-05" />
-      </inertial>
-      <visual>
-        <origin
-          xyz="0 0 0"
-          rpy="0 0 0" />
-        <geometry>
-          <mesh
-            filename="package://bobac3_description/meshes/top_camera_link.STL" />
-        </geometry>
-        <material
-          name="">
-          <color
-            rgba="0.5 0.5 0.5 1" />
-        </material>
-      </visual>
-      <collision>
-        <origin
-          xyz="0 0 0"
-          rpy="0 0 0" />
-        <geometry>
-          <mesh
-            filename="package://bobac3_description/meshes/top_camera_link.STL" />
-        </geometry>
-      </collision>
-    </link>
-    <joint name="top_camera_joint" type="fixed">
-      <origin
-        xyz="0.039197 0 0.446233"
-        rpy="0 -0.314159 0" />
+          xyz="0.039197 0 0.446233"
+          rpy="0 -0.314159 0" />
+      </xacro:unless>
       <parent
         link="basic_kit_link" />

File: src/bobac3_description/xacro/bobac3_base.xacro (robot description, xacro)
@@ -7,22 +7,22 @@
   <xacro:property name="black" value="1 1 1 1" />
   <!-- 宏 -->
-  <xacro:macro name="bobac3_body" params="sim">
+  <xacro:macro name="bobac3_body" params="sim laser_type">
     <link name="base_footprint">
       <visual>
         <origin xyz="0.0 0.0 0.0" rpy="0.0 0.0 0.0" />
         <geometry>
-          <cylinder radius="0.001" length="0.001" />
+          <cylinder radius="0.12" length="0.025" />
         </geometry>
         <material name="LightGrey">
-          <color rgba="1.0 1.0 1.0 0.0" />
-        </material>
-      </visual>
-      <collision>
-        <geometry>
-          <cylinder radius="0.15" length="0.01" />
+          <color rgba="1.0 1.0 1.0 1.0" />
+        </material>
+      </visual>
+      <collision>
+        <geometry>
+          <cylinder radius="0.12" length="0.025" />
         </geometry>
       </collision>
       <inertial>
-        <mass value="500.0" />
+        <mass value="5.0" />
         <origin xyz="0.0 0.0 0.0" rpy="0.0 0.0 0.0" />
         <inertia ixx="3.0" ixy="0.0" ixz="0.0" iyy="3.0" iyz="0.0" izz="3.0" />
@@ -32,5 +32,5 @@
       <!-- xyz="0.0 0 0.03" -->
       <origin
-        xyz="0.0 0 0.005"
+        xyz="0.0 0 0.0125"
         rpy="0 0 0" />
       <parent link="base_footprint" />
@@ -372,50 +372,101 @@
       <origin xyz="0 0 0" rpy="-1.57079 0 -1.57079" />
     </joint>
-    <link
-      name="cover_link">
-      <inertial>
-        <origin
-          xyz="-0.046031 0.00010977 -0.012195"
-          rpy="0 0 0" />
-        <mass
-          value="0.02" />
-        <inertia
-          ixx="0.00774898970484328"
-          ixy="-3.1152804546131E-05"
-          ixz="0.00121855966116614"
-          iyy="0.0118594846218277"
-          iyz="1.4019804830066E-05"
-          izz="0.01764520183544" />
-      </inertial>
-      <visual>
-        <origin
-          xyz="0 0 0"
-          rpy="0 0 0" />
-        <geometry>
-          <mesh
-            filename="package://bobac3_description/meshes/cover_link.STL" />
-        </geometry>
-        <material
-          name="">
-          <color
-            rgba="0.3 0.3 0.3 1" />
-        </material>
-      </visual>
-      <collision>
-        <origin
-          xyz="0 0 0"
-          rpy="0 0 0" />
-        <geometry>
-          <mesh
-            filename="package://bobac3_description/meshes/cover_link.STL" />
-        </geometry>
-      </collision>
-    </link>
+    <xacro:if value="${laser_type == 'CSPC'}">
+      <link
+        name="cover_link">
+        <inertial>
+          <origin
+            xyz="-0.0354525819847529 0.00107783094708411 -0.0198121193715805"
+            rpy="0 0 0" />
+          <mass
+            value="0.944663417652184" />
+          <inertia
+            ixx="0.00528140559371182"
+            ixy="3.26493500090459E-07"
+            ixz="2.25237877582117E-07"
+            iyy="0.00753457964508637"
+            iyz="3.39315515029986E-07"
+            izz="0.0127694070178216" />
+        </inertial>
+        <visual>
+          <origin
+            xyz="0 0 0"
+            rpy="0 0 0" />
+          <geometry>
+            <mesh
+              filename="package://bobac3_description/meshes/cover_link_cspc.STL" />
+          </geometry>
+          <material
+            name="">
+            <color
+              rgba="1 1 1 1" />
+          </material>
+        </visual>
+        <collision>
+          <origin
+            xyz="0 0 0"
+            rpy="0 0 0" />
+          <geometry>
+            <mesh
+              filename="package://bobac3_description/meshes/cover_link_cspc.STL" />
+          </geometry>
+        </collision>
+      </link>
+    </xacro:if>
+    <xacro:unless value="${laser_type == 'CSPC'}">
+      <link
+        name="cover_link">
+        <inertial>
+          <origin
+            xyz="-0.046031 0.00010977 -0.012195"
+            rpy="0 0 0" />
+          <mass
+            value="0.02" />
+          <inertia
+            ixx="0.00774898970484328"
+            ixy="-3.1152804546131E-05"
+            ixz="0.00121855966116614"
+            iyy="0.0118594846218277"
+            iyz="1.4019804830066E-05"
+            izz="0.01764520183544" />
+        </inertial>
+        <visual>
+          <origin
+            xyz="0 0 0"
+            rpy="0 0 0" />
+          <geometry>
+            <mesh
+              filename="package://bobac3_description/meshes/cover_link.STL" />
+          </geometry>
+          <material
+            name="">
+            <color
+              rgba="0.3 0.3 0.3 1" />
+          </material>
+        </visual>
+        <collision>
+          <origin
+            xyz="0 0 0"
+            rpy="0 0 0" />
+          <geometry>
+            <mesh
+              filename="package://bobac3_description/meshes/cover_link.STL" />
+          </geometry>
+        </collision>
+      </link>
+    </xacro:unless>
     <joint
       name="cover_joint"
       type="fixed">
-      <origin
-        xyz="0.034465 0 0.2945"
-        rpy="0 0 0" />
+      <xacro:if value="${laser_type == 'CSPC'}">
+        <origin
+          xyz="0.042015 0 0.2945"
+          rpy="0 0 0" />
+      </xacro:if>
+      <xacro:unless value="${laser_type == 'CSPC'}">
+        <origin
+          xyz="0.034465 0 0.2945"
+          rpy="0 0 0" />
+      </xacro:unless>
       <parent
         link="base_link" />
@@ -481,20 +532,68 @@
       <origin xyz="0 0 0" rpy="0 0 0" />
     </joint>
-    <link name="front_lidar_link">
-      <inertial>
-        <origin
-          xyz="0.00651720558030218 0.000224562408974172 -0.00112325450691295"
-          rpy="0 0 0" />
-        <mass
-          value="0.0887019460026471" />
-        <inertia
-          ixx="2.80379133598153E-05"
-          ixy="2.93497586302144E-07"
-          ixz="7.72249383101937E-06"
-          iyy="5.04302779195181E-05"
-          iyz="-1.22728007694022E-07"
-          izz="5.59356812720871E-05" />
-      </inertial>
-      <visual>
+    <xacro:if value="${laser_type == 'CSPC'}">
+      <link
+        name="front_lidar_link">
+        <inertial>
+          <origin
+            xyz="9.79620733382314E-06 3.84424463006512E-05 0.0154349889563586"
+            rpy="0 0 0" />
+          <mass
+            value="0.0149704923132453" />
+          <inertia
+            ixx="2.47304432946628E-06"
+            ixy="-1.99227965010988E-08"
+            ixz="-1.34962913459216E-09"
+            iyy="2.41977759114989E-06"
+            iyz="-4.87056711198406E-09"
+            izz="4.36283158743968E-06" />
+        </inertial>
+        <visual>
+          <origin
+            xyz="0 0 0"
+            rpy="0 0 0" />
+          <geometry>
+            <mesh
+              filename="package://bobac3_description/meshes/front_lidar_link_cspc.STL" />
+          </geometry>
+          <material
+            name="">
+            <color
+              rgba="0 0 0.7 1" />
+          </material>
+        </visual>
+      </link>
+    </xacro:if>
+    <xacro:unless value="${laser_type == 'CSPC'}">
+      <link name="front_lidar_link">
+        <inertial>
+          <origin
+            xyz="0.00651720558030218 0.000224562408974172 -0.00112325450691295"
+            rpy="0 0 0" />
+          <mass
+            value="0.0887019460026471" />
+          <inertia
+            ixx="2.80379133598153E-05"
+            ixy="2.93497586302144E-07"
+            ixz="7.72249383101937E-06"
+            iyy="5.04302779195181E-05"
+            iyz="-1.22728007694022E-07"
+            izz="5.59356812720871E-05" />
+        </inertial>
+        <visual>
+          <origin
+            xyz="0 0 0"
+            rpy="0 0 0" />
+          <geometry>
+            <mesh
+              filename="package://bobac3_description/meshes/front_lidar_link.STL" />
+          </geometry>
+          <material
+            name="">
+            <color
+              rgba="0 0 0.7 1" />
+          </material>
+        </visual>
+        <!-- <collision>
         <origin
           xyz="0 0 0"
@@ -504,24 +603,18 @@
             filename="package://bobac3_description/meshes/front_lidar_link.STL" />
         </geometry>
-        <material
-          name="">
-          <color
-            rgba="0 0 0.7 1" />
-        </material>
-      </visual>
-      <!-- <collision>
-      <origin
-        xyz="0 0 0"
-        rpy="0 0 0" />
-      <geometry>
-        <mesh
-          filename="package://bobac3_description/meshes/front_lidar_link.STL" />
-      </geometry>
-    </collision> -->
-    </link>
+      </collision> -->
+      </link>
+    </xacro:unless>
     <joint name="base_front_lidar_joint" type="fixed">
-      <origin
-        xyz="0.140504013961284 0 0.217"
-        rpy="3.14159265358979 0 1.5707963267949" />
+      <xacro:if value="${laser_type == 'CSPC'}">
+        <origin
+          xyz="0.13952 5.5671E-05 0.20816"
+          rpy="0 0 0" />
+      </xacro:if>
+      <xacro:unless value="${laser_type == 'CSPC'}">
+        <origin
+          xyz="0.140504013961284 0 0.217"
+          rpy="3.14159265358979 0 1.5707963267949" />
+      </xacro:unless>
       <parent
         link="base_link" />
@@ -531,20 +624,68 @@
         xyz="0 0 0" />
     </joint>
-    <link name="rear_lidar_link">
-      <inertial>
-        <origin
-          xyz="0.0065172055803022 0.000224562408974144 -0.00112325450691295"
-          rpy="0 0 0" />
-        <mass
-          value="0.088701946002647" />
-        <inertia
-          ixx="2.80379133598153E-05"
-          ixy="2.93497586302134E-07"
-          ixz="7.72249383101936E-06"
-          iyy="5.04302779195181E-05"
-          iyz="-1.22728007694019E-07"
-          izz="5.59356812720871E-05" />
-      </inertial>
-      <visual>
+    <xacro:if value="${laser_type == 'CSPC'}">
+      <link
+        name="rear_lidar_link">
+        <inertial>
+          <origin
+            xyz="9.77370904767239E-06 9.40515125694615E-05 0.0154371252989986"
+            rpy="0 0 0" />
+          <mass
+            value="0.014970492367833" />
+          <inertia
+            ixx="2.47304419700334E-06"
+            ixy="-1.99229697216871E-08"
+            ixz="-1.34960286394679E-09"
+            iyy="2.41977744844693E-06"
+            iyz="-4.87056453682969E-09"
+            izz="4.36283125537936E-06" />
+        </inertial>
+        <visual>
+          <origin
+            xyz="0 0 0"
+            rpy="0 0 0" />
+          <geometry>
+            <mesh
+              filename="package://bobac3_description/meshes/rear_lidar_link_cspc.STL" />
+          </geometry>
+          <material
+            name="">
+            <color
+              rgba="0 0 0.7 1" />
+          </material>
+        </visual>
+      </link>
+    </xacro:if>
+    <xacro:unless value="${laser_type == 'CSPC'}">
+      <link name="rear_lidar_link">
+        <inertial>
+          <origin
+            xyz="0.0065172055803022 0.000224562408974144 -0.00112325450691295"
+            rpy="0 0 0" />
+          <mass
+            value="0.088701946002647" />
+          <inertia
+            ixx="2.80379133598153E-05"
+            ixy="2.93497586302134E-07"
+            ixz="7.72249383101936E-06"
+            iyy="5.04302779195181E-05"
+            iyz="-1.22728007694019E-07"
+            izz="5.59356812720871E-05" />
+        </inertial>
+        <visual>
+          <origin
+            xyz="0 0 0"
+            rpy="0 0 0" />
+          <geometry>
+            <mesh
+              filename="package://bobac3_description/meshes/rear_lidar_link.STL" />
+          </geometry>
+          <material
+            name="">
+            <color
+              rgba="0 0 0.7 1" />
+          </material>
+        </visual>
+        <!-- <collision>
         <origin
           xyz="0 0 0"
@@ -554,26 +695,20 @@
             filename="package://bobac3_description/meshes/rear_lidar_link.STL" />
         </geometry>
-        <material
-          name="">
-          <color
-            rgba="0 0 0.7 1" />
-        </material>
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
File: src/bobac3_description/xacro/bobac3_serverbot.xacro (robot description, xacro)
@@ -3,6 +3,7 @@
   <xacro:include filename="$(find bobac3_description)/xacro/bobac3_base.xacro"/>
   <xacro:include filename="$(find bobac3_description)/xacro/basic_kit.xacro"/>
+  <xacro:arg name="laser_type" default="CSPC" />
   <xacro:arg name="sim" default="0" />
-  <xacro:bobac3_body sim="$(arg sim)"/>
-  <xacro:basic_kit parent="cover_link" xyz="-0.034 0 0" rpy="0 0 0" sim="$(arg sim)"/>
+  <xacro:bobac3_body sim="$(arg sim)" laser_type="$(arg laser_type)"/>
+  <xacro:basic_kit parent="cover_link" sim="$(arg sim)" laser_type="$(arg laser_type)"/>
 </robot>
