Commit message: awdwa

File: src/bobac3_description/xacro/gazebo_plugin.xacro (robot description, xacro)
@@ -16,11 +16,9 @@
     <gazebo reference="base_footprint">
       <material>Gazebo/GreyTransparent</material>
-      <mu1>0.0</mu1>
-      <mu2>0.0</mu2>
     </gazebo>
     <gazebo reference="base_link">
       <material>Gazebo/White</material>
     </gazebo>
-    <gazebo reference="humtmper_link">
+    <gazebo reference="humtemper_link">
       <material>Gazebo/FlatBlack</material>
     </gazebo>
@@ -34,5 +32,5 @@
       <material>Gazebo/FlatBlack</material>
     </gazebo>
-    <gazebo reference="smoke_link">
+    <gazebo reference="smoke_sensor_link">
       <material>Gazebo/FlatBlack</material>
     </gazebo>
@@ -49,19 +47,4 @@
       <material>Gazebo/FlatBlack</material>
     </gazebo>
-    <gazebo reference="left/wheel_link">
-      <material>Gazebo/FlatBlack</material>
-      <mu1>0.0</mu1>
-      <mu2>0.0</mu2>
-    </gazebo>
-    <gazebo reference="right/wheel_link">
-      <material>Gazebo/FlatBlack</material>
-      <mu1>0.0</mu1>
-      <mu2>0.0</mu2>
-    </gazebo>
-    <gazebo reference="front/wheel_link">
-      <material>Gazebo/FlatBlack</material>
-      <mu1>0.0</mu1>
-      <mu2>0.0</mu2>
-    </gazebo>
     <gazebo reference="fuse_lidar_link">
       <material>Gazebo/BlueLaser</material>
@@ -69,10 +52,10 @@
         <pose>0 0 0 0 0 0</pose>
         <visualize>false</visualize>
-        <update_rate>20</update_rate>
+        <update_rate>10</update_rate>
         <ray>
           <scan>
             <horizontal>
               <samples>720</samples>
-              <resolution>0.5</resolution>
+              <resolution>1</resolution>
               <min_angle>-3.14159</min_angle>
               <max_angle>3.14159</max_angle>
@@ -81,5 +64,5 @@
           <range>
             <min>0.15</min>
-            <max>10.0</max>
+            <max>30.0</max>
             <resolution>0.01</resolution>
           </range>
@@ -187,24 +170,4 @@
       </sensor>
     </gazebo>
-    <gazebo reference="base_footprint">
-      <gravity>true</gravity>
-      <sensor name="imu_sensor" type="imu">
-        <always_on>true</always_on>
-        <update_rate>100</update_rate>
-        <visualize>true</visualize>
-        <topic>/imu_data</topic>
-        <plugin filename="libgazebo_ros_imu_sensor.so" name="imu_plugin">
-          <topicName>/imu</topicName>
-          <bodyName>base_footprint</bodyName>
-          <updateRateHZ>100.0</updateRateHZ>
-          <gaussianNoise>0.0</gaussianNoise>
-          <xyzOffset>0 0 0</xyzOffset>
-          <rpyOffset>0 0 0</rpyOffset>
-          <frameName>base_footprint</frameName>
-          <initialOrientationAsReference>false</initialOrientationAsReference>
-        </plugin>
-        <pose>0 0 0 0 0 0</pose>
-      </sensor>
-    </gazebo>
   </xacro:macro>
 </robot>
